Commit message: fix wr3 collision

File: assets/wr3/wr3.urdf (robot description, URDF)
Before this commit: robot wr3, 14 links, 13 joints
Links:
- link FL_calf_link: geometry collision mesh filename=./meshes/FL_calf_link.STL; visual mesh filename=./meshes/FL_calf_link.STL
- link FL_hip_link: geometry visual mesh filename=./meshes/FL_hip_link.STL
- link FL_thigh_link: geometry visual mesh filename=./meshes/FL_thigh_link.STL
- link FR_calf_link: geometry collision mesh filename=./meshes/FR_calf_link.STL; visual mesh filename=./meshes/FR_calf_link.STL
- link FR_hip_link: geometry visual mesh filename=./meshes/FR_hip_link.STL
- link FR_thigh_link: geometry visual mesh filename=./meshes/FR_thigh_link.STL
- link RL_calf_link: geometry collision mesh filename=./meshes/RL_calf_link.STL; visual mesh filename=./meshes/RL_calf_link.STL
- link RL_hip_link: geometry visual mesh filename=./meshes/RL_hip_link.STL
- link RL_thigh_link: geometry visual mesh filename=./meshes/RL_thigh_link.STL
- link RR_calf_link: geometry collision mesh filename=./meshes/RR_calf_link.STL; visual mesh filename=./meshes/RR_calf_link.STL
- link RR_hip_link: geometry visual mesh filename=./meshes/RR_hip_link.STL
- link RR_thigh_link: geometry visual mesh filename=./meshes/RR_thigh_link.STL
- link trunk_link: geometry collision mesh filename=./meshes/trunk_link.STL; visual mesh filename=./meshes/trunk_link.STL

Commit message: add urdf self collision filter

File: assets/wr3/wr3.urdf (robot description, URDF)
Before this commit: robot wr3, 14 links, 13 joints
Links:
- link FL_hip_link: geometry collision mesh filename=./meshes/FL_hip_link.STL; visual mesh filename=./meshes/FL_hip_link.STL
- link FL_thigh_link: geometry collision mesh filename=./meshes/FL_thigh_link.STL; visual mesh filename=./meshes/FL_thigh_link.STL
- link FR_hip_link: geometry collision mesh filename=./meshes/FR_hip_link.STL; visual mesh filename=./meshes/FR_hip_link.STL
- link FR_thigh_link: geometry collision mesh filename=./meshes/FR_thigh_link.STL; visual mesh filename=./meshes/FR_thigh_link.STL
- link RL_hip_link: geometry collision mesh filename=./meshes/RL_hip_link.STL; visual mesh filename=./meshes/RL_hip_link.STL
- link RL_thigh_link: geometry collision mesh filename=./meshes/RL_thigh_link.STL; visual mesh filename=./meshes/RL_thigh_link.STL
- link RR_hip_link: geometry collision mesh filename=./meshes/RR_hip_link.STL; visual mesh filename=./meshes/RR_hip_link.STL
- link RR_thigh_link: geometry collision mesh filename=./meshes/RR_thigh_link.STL; visual mesh filename=./meshes/RR_thigh_link.STL
